File: core.brd (EAGLE design)
At the start: 131.8 x 142.2 mm, 279 parts, among them IC1 MAX481CSA, IC10 MAX481CSA, IC11 MAX481CSA, IC12 MAX481CSA, IC13 MAX481CSA, IC14 MAX481CSA, IC15 MAX481CSA, IC16 MAX481CSA, IC17 MAX481CSA, IC18 MAX481CSA, IC19 MAX481CSA, IC2 LD117AS12TR, IC20 MAX481CSA, IC21 MAX481CSA, IC3 MAX481CSA, IC4 MAX481CSA, IC5 MAX481CSA, IC6 MAX481CSA, IC7 MAX481CSA, IC8 MAX481CSA, IC9 MAX481CSA

Commit message: Core 001 Complete
Parts:
- moved JTAG 36.3 mm to (122.6, 23.5)
- moved ACCESSORY_GPIO 34.9 mm to (84.5, 31.1)
- moved ACCESSORY 17.9 mm to (102.9, 31.1)
- moved H2 4.44 mm to (127.0, 132.7)
- moved H3 4.44 mm to (5.08, 132.7)
- moved LEDARRAY 3.70 mm to (122.6, 47.6)
- moved NEBULA_H 1.27 mm to (95.9, 50.8)
- moved ULN1 1.27 mm to (122.6, 62.2)
- moved C34 1.27 mm to (87.6, 48.9)
Routing:
- net G12: track 75.0 -> 135.5 mm
- net 14: track 55.5 -> 110.1 mm, vias 1 -> 0
- net 36: track 111.2 -> 162.5 mm, vias 1 -> 2
- net 15: track 66.7 -> 107.4 mm
- net D7: track 55.5 -> 94.9 mm
- net 17: track 376.2 -> 340.5 mm, vias 5 -> 6
- net A15: track 64.1 -> 99.7 mm
- net 32: track 135.7 -> 104.3 mm, vias 3 -> 1
- net 25: track 129.9 -> 99.3 mm, vias 1 -> 2
- net 27: track 103.7 -> 133.9 mm
- net +12V: track 126.4 -> 98.4 mm, vias 2 -> 1
- net 12: track 62.5 -> 89.1 mm, vias 1 -> 0
- net N$148: track 39.7 -> 66.0 mm
- net D11: track 60.0 -> 85.7 mm, vias 1 -> 2
- net E13: track 36.7 -> 60.2 mm, vias 2 -> 1
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Other:
- board size 131.8 x 142.2 mm -> 131.8 x 137.8 mm
- board text removed: "NOVA CORE v001 jm@casler.org"
