File: hardware/core/build_002/core.brd (EAGLE design)
At the start: 131.8 x 142.2 mm, 279 parts, among them IC1 MAX481CSA, IC10 MAX481CSA, IC11 MAX481CSA, IC12 MAX481CSA, IC13 MAX481CSA, IC14 MAX481CSA, IC15 MAX481CSA, IC16 MAX481CSA, IC17 MAX481CSA, IC18 MAX481CSA, IC19 MAX481CSA, IC2 LD117AS12TR, IC20 MAX481CSA, IC21 MAX481CSA, IC3 MAX481CSA, IC4 MAX481CSA, IC5 MAX481CSA, IC6 MAX481CSA, IC7 MAX481CSA, IC8 MAX481CSA, IC9 MAX481CSA

Commit message: v002
Parts:
- added JP1: (no value), pinhead:1X02
Connections:
- net 13: now also JP1.1
- net N$89: now also JP1.2
Routing:
- net GND: track 847.0 -> 750.6 mm, vias 45 -> 50
- net 17: track 376.2 -> 305.9 mm, vias 5 -> 4
- net 22/SCL: track 356.5 -> 296.7 mm, vias 8 -> 9
- net 32: track 135.7 -> 95.4 mm, vias 3 -> 2
- net +3V3: track 765.3 -> 726.2 mm, vias 8 -> 6
- net C6: track 39.2 -> 76.8 mm
- net 13: track 433.9 -> 470.0 mm, vias 9 -> 14
- net 25: track 129.9 -> 99.6 mm, vias 1 -> 2
- net D7: track 55.5 -> 85.8 mm
- net A7: track 54.2 -> 82.4 mm, vias 2 -> 1
- net E12: track 61.0 -> 35.2 mm, vias 1 -> 3
- net A6: track 62.3 -> 87.6 mm
- net B7: track 77.9 -> 52.7 mm
- net D2: track 77.3 -> 54.5 mm, vias 1 -> 2
- net G1: track 49.0 -> 27.3 mm
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Other:
- board text added: "NOVA CORE v002 jm@casler.org"
- board text added: "Nova Core v002 (c) Jm Casler 2022 www.casler.org www.oontz.com"
- board text removed: "NOVA CORE v001 jm@casler.org"
- board text removed: "Nova Core v001 (c) Jm Casler 2022 www.casler.org www.oontz.com"
