File: hardware/core/build_002/core.sch (EAGLE design)
At the start: 279 parts, among them IC1 MAX481CSA, IC10 MAX481CSA, IC11 MAX481CSA, IC12 MAX481CSA, IC13 MAX481CSA, IC14 MAX481CSA, IC15 MAX481CSA, IC16 MAX481CSA, IC17 MAX481CSA, IC18 MAX481CSA, IC19 MAX481CSA, IC2 LD117AS12TR, IC20 MAX481CSA, IC21 MAX481CSA, IC3 MAX481CSA, IC4 MAX481CSA, IC5 MAX481CSA, IC6 MAX481CSA, IC7 MAX481CSA, IC8 MAX481CSA, IC9 MAX481CSA

Commit message: v002
Parts:
- added JP1: (no value), pinhead:PINHD-1X2
Connections:
- net 13: now also JP1.1
- net N$89: now also JP1.2
Changed lines of the file:
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@@
 <part name="GND2" library="supply1" library_urn="urn:adsk.eagle:library:371" deviceset="GND" device=""/>
 <part name="+3V48" library="supply1" library_urn="urn:adsk.eagle:library:371" deviceset="+3V3" device=""/>
+<part name="JP1" library="pinhead" library_urn="urn:adsk.eagle:library:325" deviceset="PINHD-1X2" device="" package3d_urn="urn:adsk.eagle:package:22435/2"/>
 </parts>
 <sheets>
@@
 <attribute name="VALUE" x="104.14" y="-53.34" size="1.778" layer="96" rot="R270"/>
 </instance>
+<instance part="JP1" gate="G$1" x="231.14" y="-2.54" smashed="yes" rot="R180">
+<attribute name="NAME" x="237.49" y="-8.255" size="1.778" layer="95" rot="R180"/>
+<attribute name="VALUE" x="237.49" y="2.54" size="1.778" layer="96" rot="R180"/>
+</instance>
 </instances>
 <busses>
@@
 <junction x="274.32" y="-5.08"/>
 <label x="269.24" y="-12.7" size="1.778" layer="95"/>
+<pinref part="JP1" gate="G$1" pin="1"/>
+<wire x1="256.54" y1="-5.08" x2="233.68" y2="-5.08" width="0.1524" layer="91"/>
+<junction x="256.54" y="-5.08"/>
 </segment>
 </net>
@@
 <pinref part="J1" gate="G$1" pin="2"/>
 <pinref part="R68" gate="G$1" pin="1"/>
+<pinref part="JP1" gate="G$1" pin="2"/>
+<wire x1="256.54" y1="-2.54" x2="233.68" y2="-2.54" width="0.1524" layer="91"/>
+<junction x="256.54" y="-2.54"/>
 </segment>
 </net>
